Commit message: Activate cameras in sim

File: prl_ur5_description/urdf/_camera_sensor.urdf.xacro (robot description, xacro)
@@ -4,5 +4,5 @@
   <xacro:include filename="$(find realsense2_description)/urdf/_d435i.urdf.xacro"/>
   <xacro:include filename="$(find prl_ur5_description)/urdf/_d435.gazebo.xacro"/>
-  <xacro:macro name="camera_sensor" params="prefix parent camera pose">
+  <xacro:macro name="camera_sensor" params="prefix parent camera pose turn_on:=false">
     <!-- check camera type -->
     <xacro:unless value="${camera in [None, 'realsense-d435i']}">
@@ -14,5 +14,5 @@
         <origin xyz="${pose['x']} ${pose['y']} ${pose['z']}" rpy="${pose['roll']} ${pose['pitch']} ${pose['yaw']}"/>
       </xacro:sensor_d435i>
-      <xacro:gazebo_d435 name="${prefix}camera"/>
+      <xacro:gazebo_d435 name="${prefix}camera" turn_on="${turn_on}"/>
     </xacro:if>
   </xacro:macro>

File: prl_ur5_description/urdf/_d435.gazebo.xacro (robot description, xacro)
@@ -8,5 +8,5 @@
 <!-- Modified from https://github.com/pal-robotics-forks/realsense -->
 <robot xmlns:xacro="http://ros.org/wiki/xacro">
-  <xacro:macro name="gazebo_d435" params="name publish_pointcloud:=true visualize:=false" >
+  <xacro:macro name="gazebo_d435" params="name turn_on publish_pointcloud:=true visualize:=false" >
     <!-- Load parameters to model's main link-->
     <xacro:property name="deg_to_rad" value="${pi/180}" />
@@ -44,5 +44,5 @@
           </noise>
         </camera>
-        <always_on>0</always_on>
+        <always_on>${turn_on}</always_on>
         <update_rate>30</update_rate>
         <visualize>${visualize}</visualize>
@@ -109,5 +109,5 @@
           </noise>
         </camera>
-        <always_on>0</always_on>
+        <always_on>${turn_on}</always_on>
         <update_rate>90</update_rate>
         <visualize>0</visualize>

File: prl_ur5_description/urdf/_ur5.urdf.xacro (robot description, xacro)
@@ -16,4 +16,5 @@
       joint_limits
       hardware_interface
+      sensors
       gripper:=None
       gripper_pose:=None
@@ -68,5 +69,5 @@
     <!-- hand-eye camera -->
     <xacro:unless value="${camera is None}">
-      <xacro:camera_sensor camera="${camera}" prefix='${prefix}' parent="${prefix}tool" pose="${camera_pose}"/>
+      <xacro:camera_sensor camera="${camera}" prefix='${prefix}' parent="${prefix}tool" pose="${camera_pose}" turn_on="${sensors}"/>
     </xacro:unless>
   </xacro:macro>

File: prl_ur5_description/urdf/prl_ur5.urdf.xacro (robot description, xacro)
@@ -7,5 +7,5 @@
   <!-- Fixed cameras -->
   <xacro:include filename="$(find prl_ur5_description)/urdf/_fixed_cameras.urdf.xacro"/>
-  <xacro:macro name="prl_ur5" params="setup_file hardware_interface table:=true backwall:=true ceiling:=true">
+  <xacro:macro name="prl_ur5" params="setup_file hardware_interface sensors:=false table:=true backwall:=true ceiling:=true">
     <!-- base link -->
     <link name="prl_ur5_base"/>
@@ -17,6 +17,6 @@
         </geometry>
         <material name="Cyan">
-  14        <color rgba="0 1.0 1.0 1.0"/>
-  15      </material>
+          <color rgba="0 1.0 1.0 1.0"/>
+        </material>
       </visual>
       <collision>
@@ -107,4 +107,5 @@
                  gripper="${left.get('gripper')}"
                  gripper_pose="${left.get('gripper_pose')}"
+                 sensors="${sensors}"
                  camera="${left.get('camera')}"
                  camera_pose="${left.get('camera_pose')}"
@@ -121,4 +122,5 @@
                  gripper="${right.get('gripper')}"
                  gripper_pose="${right.get('gripper_pose')}"
+                 sensors="${sensors}"
                  camera="${right.get('camera')}"
                  camera_pose="${right.get('camera_pose')}"

File: prl_ur5_description/urdf/prl_ur5_robot.urdf.xacro (robot description, xacro)
@@ -4,4 +4,5 @@
   <xacro:arg name="setup" default="standart_setup"/>
   <xacro:arg name="table" default="true"/>
+  <xacro:arg name="sensors" default="false"/>
   <xacro:arg name="hardware_interface" default="hardware_interface/PositionJointInterface"/>
   <!-- ur5 robot -->
@@ -9,4 +10,5 @@
   <xacro:prl_ur5 setup_file="${xacro.load_yaml('$(find prl_ur5_robot_configuration)/config/$(arg setup).yaml')}"
                  table="$(arg table)"
-                 hardware_interface="$(arg hardware_interface)"/>
+                 hardware_interface="$(arg hardware_interface)"
+                 sensors="$(arg sensors)"/>
 </robot>

Commit message: Camera frames are automatically published from config file for real and sim robot + Update configuration file (+minor readme update)

File: prl_ur5_description/urdf/_camera_sensor.urdf.xacro (robot description, xacro)
@@ -11,5 +11,5 @@
     <!-- if realsense d435i -->
     <xacro:if value="${camera == 'realsense-d435i'}">
-      <xacro:sensor_d435i name="${prefix}camera" parent="${prefix}tool">
+      <xacro:sensor_d435i name="${prefix}camera" parent="${parent}" use_nominal_extrinsics="true">
         <origin xyz="${pose['x']} ${pose['y']} ${pose['z']}" rpy="${pose['roll']} ${pose['pitch']} ${pose['yaw']}"/>
       </xacro:sensor_d435i>

File: prl_ur5_description/urdf/_fixed_cameras.urdf.xacro (robot description, xacro)
@@ -1,21 +1,46 @@
 <?xml version="1.0"?>
 <robot xmlns:xacro="http://wiki.ros.org/xacro">
+    <!-- Including this file a second time would include 'realsense2_description/urdf/_d435i.urdf.xacro' a second time which will result in a crash related to this problem :  https://github.com/IntelRealSense/realsense-ros/issues/2338 -->
+    <!-- It is assumed that this file has already been included somewhere else (e.g. in _ur5.urdf.xacro) -->
+    <!-- <xacro:include filename="$(find prl_ur5_description)/urdf/_camera_sensor.urdf.xacro"/> -->
     <!-- Build fixed camera with their support from one file -->
-    <xacro:macro name="fixed_cameras" params="parent fixed_cameras_file">
+    <xacro:macro name="fixed_cameras" params="parent fixed_cameras_file turn_on:=false">
         <xacro:property name="fixed_cameras" value="${xacro.load_yaml(fixed_cameras_file)}"/>
-        <xacro:fixed_cameras_loop parent="${parent}" number="0" cameras="${fixed_cameras}"/>
+        <xacro:fixed_cameras_loop parent="${parent}" number="0" cameras="${fixed_cameras}" turn_on="${turn_on}"/>
     </xacro:macro>
     <!-- Reccursive macro to iterate over all the cameras -->
-    <xacro:macro name="fixed_cameras_loop" params="parent number cameras">
+    <xacro:macro name="fixed_cameras_loop" params="parent number cameras turn_on">
         <xacro:if value="${cameras}">
                 <!-- pop first item from list -->
                 <xacro:property name="camera" value="${cameras.pop(0)}"/>
-                <xacro:fixed_camera parent="${parent}" number="${number}" camera="${camera}"/>
+                <xacro:fixed_camera parent="${parent}" number="${number}" camera="${camera}" turn_on="${turn_on}"/>
                 <!-- recursively call myself -->
-                <xacro:fixed_cameras_loop parent="${parent}" number="${number+1}" cameras="${cameras}"/>
+                <xacro:fixed_cameras_loop parent="${parent}" number="${number+1}" cameras="${cameras}" turn_on="${turn_on}"/>
         </xacro:if>
     </xacro:macro>
     <!-- Build one camera with its stand -->
-    <xacro:macro name="fixed_camera" params="parent number camera">
+    <xacro:macro name="fixed_camera" params="parent number camera turn_on">
+        <!-- Spawn camera -->
+            <!-- check camera type -->
+        <xacro:unless value="${camera['type'] in ['realsense-d435i']}">
+            <xacro:unknown_camera_type/>
+        </xacro:unless>
+            <!-- if realsense d435i -->
+        <xacro:if value="${camera['type'] == 'realsense-d435i'}">
+            <link name="${camera['name_prefix']}_camera_calibration_pose"/>
+            <joint name="${camera['name_prefix']}_camera_calibration_pose_joint" type="fixed">
+                <origin xyz="${camera['pose']['x']} ${camera['pose']['y']} ${camera['pose']['z']}" rpy="${camera['pose']['roll']} ${camera['pose']['pitch']} ${camera['pose']['yaw']}"/>
+                <parent link="${parent}"/>
+                <child link="${camera['name_prefix']}_camera_calibration_pose"/>
+            </joint>
+            <!-- This transform 'undo' the base_screw > color_optical frame transform so the image is aligned with the calibration
+            (it comes from realsense2_description/urdf/_d435.urdf.xacro) -->
+            <xacro:camera_sensor camera="${camera['type']}"
+                                 prefix="${camera['name_prefix']}_"
+                                 parent="${camera['name_prefix']}_camera_calibration_pose"
+                                 turn_on="${turn_on}"
+                                 pose="${dict(x=0.0325, y=0.0125, z=-0.0106, roll=pi/2.0, pitch=-pi/2.0, yaw=0)}"
+                                />
+        </xacro:if>
         <!-- Numerical dimensions for the fixtures -->
         <xacro:property name="extrusion_width" value="${0.045 +0.06}"/> <!-- +/-3cm margin on the real size -->
@@ -26,5 +51,5 @@
         <!-- The arbitrary values 0.92 0.92 0.29 0.52 correspond to the dimensions of the table with 1cm margin, so the extrusions are not touching the table-->
         <xacro:if value="${camera['fixture_orientation'] == '+x'}">
-            <xacro:property name="hr_len" value="${camera['position']['x'] - camera['offset']['x'] + extrusion_width/2. - 0.92}"/>
+            <xacro:property name="hr_len" value="${camera['pose']['x'] - camera['offset']['x'] + extrusion_width/2. - 0.92}"/>
             <xacro:property name="hr_x_pos_relative" value="${- hr_len/2. + extrusion_width/2.}"/>
             <xacro:property name="hr_y_pos_relative" value="0"/>
@@ -32,5 +57,5 @@
         </xacro:if>
         <xacro:if value="${camera['fixture_orientation'] == '-x'}">
-            <xacro:property name="hr_len" value="${-camera['position']['x'] + camera['offset']['x'] + extrusion_width/2. - 0.92}"/>
+            <xacro:property name="hr_len" value="${-camera['pose']['x'] + camera['offset']['x'] + extrusion_width/2. - 0.92}"/>
             <xacro:property name="hr_x_pos_relative" value="${hr_len/2. - extrusion_width/2.}"/>
             <xacro:property name="hr_y_pos_relative" value="0"/>
@@ -38,5 +63,5 @@
         </xacro:if>
         <xacro:if value="${camera['fixture_orientation'] == '+y'}">
-            <xacro:property name="hr_len" value="${camera['position']['y'] - camera['offset']['y'] + extrusion_width/2.  - 0.29}"/>
+            <xacro:property name="hr_len" value="${camera['pose']['y'] - camera['offset']['y'] + extrusion_width/2.  - 0.29}"/>
             <xacro:property name="hr_x_pos_relative" value="0"/>
             <xacro:property name="hr_y_pos_relative" value="${- hr_len/2. + extrusion_width/2.}"/>
@@ -44,34 +69,41 @@
         </xacro:if>
         <xacro:if value="${camera['fixture_orientation'] == '-y'}">
-            <xacro:property name="hr_len" value="${-camera['position']['y'] + camera['offset']['y'] + extrusion_width/2.  - 0.52}"/>
+            <xacro:property name="hr_len" value="${-camera['pose']['y'] + camera['offset']['y'] + extrusion_width/2.  - 0.52}"/>
             <xacro:property name="hr_x_pos_relative" value="0"/>
             <xacro:property name="hr_y_pos_relative" value="${hr_len/2. - extrusion_width/2.}"/>
             <xacro:property name="hr_z_rot_relative" value="-1.570796327"/>
         </xacro:if>
-        <xacro:property name="vt_len" value="${camera['position']['z'] - camera['offset']['z'] - hr_z_pos_absolute}"/>
-        <!-- Camera -->
-        <link name="fixed_camera_${number}">
+        <xacro:property name="vt_len" value="${camera['pose']['z'] - camera['offset']['z'] - hr_z_pos_absolute}"/>
+        <!-- Camera bounding box -->
+        <link name="fixed_camera_${number}_bb">
             <visual>
                 <geometry>
-                    <cylinder radius="${camera['size']['width']/2.}" length="${camera['size']['height']}"/>
+                    <cylinder radius="${camera['bounding_box']['width']/2.}" length="${camera['bounding_box']['height']}"/>
                 </geometry>
-                <material name="purple"><color rgba="0.01 0.32 0.41 1"/></material>
+                <material name="purple"><color rgba="0.01 0.32 0.41 0.1"/></material>
             </visual>
             <collision>
                 <geometry>
-                    <cylinder radius="${camera['size']['width']/2.}" length="${camera['size']['height']}"/>
+                    <cylinder radius="${camera['bounding_box']['width']/2.}" length="${camera['bounding_box']['height']}"/>
                 </geometry>
             </collision>
         </link>
-        <gazebo reference="fixed_camera_${number}">
-                <material>Gazebo/BlueGlow</material>
+        <gazebo reference="fixed_camera_${number}_bb">
+            <visual>
+            <material>
+                <ambient>0.1 0.5 0.5 0.2</ambient>
+                <diffuse>0.1 0.5 0.1 0.2</diffuse>
+                <specular>0.1 0.1 0.1 0.2</specular>
+                <emissive>0.0 0.0 0.0 0.0</emissive>
+            </material>
+            </visual>
         </gazebo>
-        <joint name="fixed_camera_${number}_fix" type="fixed">
+        <joint name="fixed_camera_${number}_bb_joint" type="fixed">
             <parent link = "${parent}"/>
-            <child link="fixed_camera_${number}"/>
-            <origin xyz="${camera['position']['x']} ${camera['position']['y']} ${camera['position']['z']}" rpy="0 0 0"/>
+            <child link="fixed_camera_${number}_bb"/>
+            <origin xyz="${camera['pose']['x']} ${camera['pose']['y']} ${camera['pose']['z']}" rpy="0 0 0"/>
         </joint>
         <!-- Spherical joint holding the camera -->
-        <link name="fixed_sj_${number}">
+        <link name="fixed_camera_${number}_sj">
             <visual>
                 <geometry>
@@ -86,14 +118,14 @@
             </collision>
         </link>
-        <gazebo reference="fixed_sj_${number}">
+        <gazebo reference="fixed_camera_${number}_sj">
                 <material>Gazebo/BlueGlow</material>
         </gazebo>
-        <joint name="fixed_sj_${number}_fix" type="fixed">
-            <parent link = "fixed_camera_${number}"/>
-            <child link="fixed_sj_${number}"/>
-            <origin xyz="0 0 ${- camera['size']['height']/2. - sj_height/2.}" rpy="0 0 0"/>
+        <joint name="fixed_camera_${number}_sj_joint" type="fixed">
+            <parent link = "fixed_camera_${number}_bb"/>
+            <child link="fixed_camera_${number}_sj"/>
+            <origin xyz="0 0 ${- camera['bounding_box']['height']/2. - sj_height/2.}" rpy="0 0 0"/>
         </joint>
         <!-- Vertical extrusion -->
-        <link name="fixed_vt_${number}">
+        <link name="fixed_camera_${number}_vt">
             <visual>
                 <geometry>
@@ -108,11 +140,11 @@
             </collision>
         </link>
-        <gazebo reference="fixed_vt_${number}">
+        <gazebo reference="fixed_camera_${number}_vt">
                 <material>Gazebo/BlueGlow</material>
         </gazebo>
-        <joint name="fixed_vt_${number}_fix" type="fixed">
-            <parent link = "fixed_sj_${number}"/>
-            <child link="fixed_vt_${number}"/>
-            <origin xyz="${-camera['offset']['x']} ${-camera['offset']['y']} ${sj_height/2. + camera['size']['height']/2. - camera['offset']['z'] - vt_len/2.}" rpy="0 0 0"/>
+        <joint name="fixed_camera_${number}_vt_joint" type="fixed">
+            <parent link = "fixed_camera_${number}_sj"/>
+            <child link="fixed_camera_${number}_vt"/>
+            <origin xyz="${-camera['offset']['x']} ${-camera['offset']['y']} ${sj_height/2. + camera['bounding_box']['height']/2. - camera['offset']['z'] - vt_len/2.}" rpy="0 0 0"/>
         </joint>
         <!-- Horizontal extrusion -->
@@ -134,5 +166,5 @@
         </gazebo>
         <joint name="fixed_hr_${number}_fix" type="fixed">
-            <parent link = "fixed_vt_${number}"/>
+            <parent link = "fixed_camera_${number}_vt"/>
             <child link="fixed_hr_${number}"/>
             <origin xyz="${hr_x_pos_relative} ${hr_y_pos_relative} ${- vt_len/2. - extrusion_width/2.}" rpy="0 0 ${hr_z_rot_relative}"/>

File: prl_ur5_description/urdf/prl_ur5.urdf.xacro (robot description, xacro)
@@ -53,5 +53,5 @@
     <!-- Cameras fixtures (if any) -->
     <xacro:if value="${setup_file.get('fixed_cameras_file') is not None}">
-      <xacro:fixed_cameras parent="prl_ur5_base" fixed_cameras_file="$(find prl_ur5_robot_configuration)/config/${setup_file['fixed_cameras_file']}"/>
+      <xacro:fixed_cameras parent="prl_ur5_base" fixed_cameras_file="$(find prl_ur5_robot_configuration)/config/${setup_file['fixed_cameras_file']}" turn_on="${sensors}"/>
     </xacro:if>
     <!-- back wall -->

File: prl_ur5_moveit_config/config/standart_setup/prl_ur5_robot.srdf.xacro (robot description, xacro)
@@ -60,5 +60,5 @@
     <xacro:call macro="${right_gripper_name}_col_with" prefix='right_gripper' link='right_ft300_mounting_plate'/>
     <xacro:call macro="${right_gripper_name}_col_with" prefix='right_gripper' link='right_ft300_sensor'/>
-    <xacro:if value="${'caemra' in setup['right']}">
+    <xacro:if value="${'camera' in setup['right']}">
         <xacro:call macro="${right_gripper_name}_col_with" prefix='right_gripper' link='right_camera_link'/>
     </xacro:if>
@@ -194,3 +194,26 @@
     <disable_collisions link1="right_wrist_2_link" link2="right_wrist_3_link" reason="Adjacent"/>
     <disable_collisions link1="right_wrist_3_link" link2="right_wrist_connector_link" reason="Adjacent"/>
+    <!-- External cameras -->
+    <xacro:macro name="external_camera_col" params="number camera">
+        <disable_collisions link1="fixed_camera_${number}_bb" link2="fixed_camera_${number}_sj" reason="Adjacent"/>
+        <disable_collisions link1="fixed_camera_${number}_vt" link2="fixed_camera_${number}_sj" reason="Adjacent"/>
+        <disable_collisions link1="fixed_camera_${number}_vt" link2="fixed_hr_${number}" reason="Adjacent"/>
+        <disable_collisions link1="fixed_camera_${number}_vt" link2="fixed_camera_${number}_bb" reason="Adjacent"/>
+        <disable_collisions link1="${camera['name_prefix']}_camera_link" link2="fixed_camera_${number}_vt" reason="Adjacent"/>
+        <disable_collisions link1="${camera['name_prefix']}_camera_link" link2="fixed_camera_${number}_sj" reason="Adjacent"/>
+        <disable_collisions link1="${camera['name_prefix']}_camera_link" link2="fixed_camera_${number}_bb" reason="Adjacent"/>
+    </xacro:macro>
+    <!-- Iterate voer all cameras using reccursive function-->
+    <xacro:property name="fixed_cameras_file" value="$(find prl_ur5_robot_configuration)/config/${setup['fixed_cameras_file']}"/>
+    <xacro:property name="fixed_cameras" value="${xacro.load_yaml(fixed_cameras_file)}"/>
+    <xacro:macro name="external_cameras_loop" params="cameras number">
+        <xacro:if value="${cameras}">
+                <!-- pop first item from list -->
+                <xacro:property name="camera" value="${cameras.pop(0)}"/>
+                <xacro:external_camera_col number="${number}" camera="${camera}"/>
+                <!-- recursive call -->
+                <xacro:external_cameras_loop cameras="${cameras}" number="${number+1}"/>
+        </xacro:if>
+    </xacro:macro>
+    <xacro:external_cameras_loop cameras="${fixed_cameras}" number="0"/>
 </robot>
