Commit message: Add connector model

File: prl_ur5_description/urdf/_ur5.urdf.xacro (robot description, xacro)
@@ -46,4 +46,23 @@
     <xacro:unless value="${gripper is None}">
       <xacro:gripper gripper="${gripper}" prefix='${prefix}' parent="${prefix}tool" pose="${gripper_pose}" hardware_interface="${hardware_interface}"/>
+      <!-- Right angle connector -->
+      <link name="${prefix}wrist_connector_link">
+        <visual>
+            <geometry>
+                <mesh filename="package://prl_ur5_description/model/RG_connector_simple.stl"/>
+            </geometry>
+            <material name="connector_green"><color rgba="0.2 0.8 0 1"/></material>
+        </visual>
+        <collision>
+            <geometry>
+                <mesh filename="package://prl_ur5_description/model/RG_connector_simple.stl"/>
+            </geometry>
+        </collision>
+      </link>
+      <joint name="${prefix}wrist_connector" type="fixed">
+        <origin xyz="0 -0.0375 -0.02" rpy="1.5708 0 0"/>
+        <parent link="${prefix}wrist_3_link"/>
+        <child link="${prefix}wrist_connector_link"/>
+      </joint>
     </xacro:unless>
     <!-- hand-eye camera -->

Commit message: CHANGE CONVENTION : GRIPPER FLIPPED 180° ON Z-AXIS. (follow original RG6 convention that cannot be bypassed anymore with v2)

File: prl_ur5_description/urdf/_ur5.urdf.xacro (robot description, xacro)
@@ -40,5 +40,5 @@
     <link name="${prefix}tool"/>
     <joint name="${prefix}tool_joint" type="fixed">
-      <origin xyz="0 0 0" rpy="0 0 0"/>
+      <origin xyz="0 0 0" rpy="0 0 ${-pi}"/>
       <parent link="${prefix}robotiq_ft_frame_id"/>
       <child link="${prefix}tool"/>

Commit message: Make remaining non convex mesh convex for collision detection : vention_tower & RG_connector_simple

File: prl_ur5_description/urdf/_ur5.urdf.xacro (robot description, xacro)
@@ -57,5 +57,5 @@
         <collision>
             <geometry>
-                <mesh filename="package://prl_ur5_description/model/RG_connector_simple.stl"/>
+                <mesh filename="package://prl_ur5_description/model/RG_connector_simple_convex.stl"/>
             </geometry>
         </collision>

File: prl_ur5_description/urdf/prl_ur5.urdf.xacro (robot description, xacro)
@@ -22,5 +22,15 @@
       <collision>
         <geometry>
-          <mesh filename="package://prl_ur5_description/model/vention_tower.stl"/>
+          <mesh filename="package://prl_ur5_description/model/vention_tower_bottom_convex.stl"/>
+        </geometry>
+      </collision>
+      <collision>
+        <geometry>
+          <mesh filename="package://prl_ur5_description/model/vention_tower_middle_convex.stl"/>
+        </geometry>
+      </collision>
+      <collision>
+        <geometry>
+          <mesh filename="package://prl_ur5_description/model/vention_tower_top_convex.stl"/>
         </geometry>
       </collision>
