Commit message: WiP: Full assembly at the right place

File: prl_ur5_description/urdf/_fixed_cameras.urdf.xacro (robot description, xacro)
@@ -18,20 +18,119 @@
     <!-- Build one camera with its stand -->
     <xacro:macro name="fixed_camera" params="parent camera">
+        <!-- Camera -->
         <link name="camera_${camera['name']}">
             <visual>
-            <geometry>
-                <box size="0.2 0.2 0.2" />
-            </geometry>
+                <geometry>
+                    <box size="${camera['size']['x']} ${camera['size']['y']} ${camera['size']['z']}" />
+                </geometry>
+                <material name="purple"><color rgba="0.8 0 0.8 1"/></material>
             </visual>
             <collision>
-            <geometry>
-                <box size="0.2 0.2 0.2" />
-            </geometry>
+                <geometry>
+                    <box size="${camera['size']['x']} ${camera['size']['y']} ${camera['size']['z']}" />
+                </geometry>
             </collision>
         </link>
+        <gazebo reference="camera_${camera['name']}">
+                <material>Gazebo/BlueGlow</material>
+        </gazebo>
         <joint name="camera_${camera['name']}_fix" type="fixed">
             <parent link = "${parent}"/>
             <child link="camera_${camera['name']}"/>
-            <origin xyz="${camera['pose']['x']} ${camera['pose']['y']} ${camera['pose']['z']}" rpy="0.0 0.0 0.0"/>
+            <origin xyz="${camera['pose']['x']} ${camera['pose']['y']} ${camera['pose']['z']}" rpy="${camera['pose']['roll']} ${camera['pose']['pitch']} ${camera['pose']['yaw']}"/>
+        </joint>
+        <!-- Numerical dimensions for the fixtures -->
+        <xacro:property name="extrusion_width" value="${0.045 +0.02}"/> <!-- +/-1cm margin on the real size -->
+        <xacro:property name="hr_z_pos" value="-0.05625"/> <!-- height at which the horizontal extrusion are fixed to the table -->
+        <xacro:property name="sj_height" value="${0.17 + 0.09}"/> <!-- Height of the spherical joint supporting the camera (plus the supporting part under) -->
+        <xacro:property name="sj_diameter" value="${0.045 +0.02}"/> <!-- Diameter of the spherical joint supporting the camera (plus the supporting part under) -->
+        <!-- Simple math to change the side of the table to which the fixture is attached-->
+        <xacro:if value="${camera['fixture_orientation'] == '+x'}">
+            <xacro:property name="hr_len" value="${camera['pose']['x'] - camera['offset']['x']}"/>
+            <xacro:property name="hr_x_pos" value="${hr_len/2.}"/>
+            <xacro:property name="hr_y_pos" value="${camera['pose']['y'] - camera['offset']['y']}"/>
+            <xacro:property name="hr_z_rot" value="0"/>
+        </xacro:if>
+        <xacro:if value="${camera['fixture_orientation'] == '-x'}">
+            <xacro:property name="hr_len" value="${-camera['pose']['x'] + camera['offset']['x']}"/>
+            <xacro:property name="hr_x_pos" value="${-hr_len/2.}"/>
+            <xacro:property name="hr_y_pos" value="${camera['pose']['y'] - camera['offset']['y']}"/>
+            <xacro:property name="hr_z_rot" value="3.1415926"/>
+        </xacro:if>
+        <xacro:if value="${camera['fixture_orientation'] == '+y'}">
+            <xacro:property name="hr_len" value="${camera['pose']['y'] - camera['offset']['y']}"/>
+            <xacro:property name="hr_x_pos" value="${camera['pose']['x'] - camera['offset']['x']}"/>
+            <xacro:property name="hr_y_pos" value="${hr_len/2.}"/>
+            <xacro:property name="hr_z_rot" value="1.570796327"/>
+        </xacro:if>
+        <xacro:if value="${camera['fixture_orientation'] == '-y'}">
+            <xacro:property name="hr_len" value="${-camera['pose']['y'] + camera['offset']['y']}"/>
+            <xacro:property name="hr_x_pos" value="${camera['pose']['x'] - camera['offset']['x']}"/>
+            <xacro:property name="hr_y_pos" value="${-hr_len/2.}"/>
+            <xacro:property name="hr_z_rot" value="-1.570796327"/>
+        </xacro:if>
+        <xacro:property name="vt_len" value="${camera['pose']['z'] - camera['offset']['z'] - hr_z_pos + extrusion_width}"/>
+        <!-- Horizontal extrusion -->
+        <link name="hr_${camera['name']}">
+            <visual>
+                <geometry>
+                    <box size="${hr_len} ${extrusion_width} ${extrusion_width}" />
+                </geometry>
+            </visual>
+            <collision>
+                <geometry>
+                    <box size="${hr_len} ${extrusion_width} ${extrusion_width}" />
+                </geometry>
+            </collision>
+        </link>
+        <gazebo reference="hr_${camera['name']}">
+                <material>Gazebo/BlueGlow</material>
+        </gazebo>
+        <joint name="hr_${camera['name']}_fix" type="fixed">
+            <parent link = "${parent}"/>
+            <child link="hr_${camera['name']}"/>
+            <origin xyz="${hr_x_pos} ${hr_y_pos} ${hr_z_pos - extrusion_width/2.}" rpy="0 0 ${hr_z_rot}"/>
+        </joint>
+        <!-- Vertical extrusion -->
+        <link name="vt_${camera['name']}">
+            <visual>
+                <geometry>
+                    <box size="${extrusion_width} ${extrusion_width} ${vt_len}" />
+                </geometry>
+            </visual>
+            <collision>
+                <geometry>
+                    <box size="${extrusion_width} ${extrusion_width} ${vt_len}" />
+                </geometry>
+            </collision>
+        </link>
+        <gazebo reference="vt_${camera['name']}">
+                <material>Gazebo/BlueGlow</material>
+        </gazebo>
+        <joint name="vt_${camera['name']}_fix" type="fixed">
+            <parent link = "${parent}"/>
+            <child link="vt_${camera['name']}"/>
+            <origin xyz="${camera['pose']['x'] - camera['offset']['x']} ${camera['pose']['y'] - camera['offset']['y']} ${camera['pose']['z']-camera['offset']['z']-vt_len/2.}" rpy="0 0 0"/>
+        </joint>
+        <!-- Spherical joint holding the camera -->
+        <link name="sj_${camera['name']}">
+            <visual>
+                <geometry>
+                    <cylinder radius="${sj_diameter/2}" length="${sj_height}"/>
+                </geometry>
+            </visual>
+            <collision>
+                <geometry>
+                    <cylinder radius="${sj_diameter/2}" length="${sj_height}"/>
+                </geometry>
+            </collision>
+        </link>
+        <gazebo reference="sj_${camera['name']}">
+                <material>Gazebo/BlueGlow</material>
+        </gazebo>
+        <joint name="sj_${camera['name']}_fix" type="fixed">
+            <parent link = "${parent}"/>
+            <child link="sj_${camera['name']}"/>
+            <origin xyz="${camera['pose']['x']} ${camera['pose']['y']} ${camera['pose']['z'] - sj_height/2.}" rpy="0 0 0"/>
         </joint>
     </xacro:macro>

File: prl_ur5_description/urdf/prl_ur5.urdf.xacro (robot description, xacro)
@@ -50,8 +50,8 @@
         <origin xyz="0.0 0.0 0.0" rpy="0.0 0.0 0.0"/>
       </joint>
-      <!-- Cameras fixtures (if any) -->
-      <xacro:if value="${setup_file.get('fixed_cameras_file') is not None}">
-        <xacro:fixed_cameras parent="prl_ur5_base" fixed_cameras_file="$(find prl_ur5_description)/config/${setup_file['fixed_cameras_file']}"/>
-      </xacro:if>
+    </xacro:if>
+    <!-- Cameras fixtures (if any) -->
+    <xacro:if value="${setup_file.get('fixed_cameras_file') is not None}">
+      <xacro:fixed_cameras parent="prl_ur5_base" fixed_cameras_file="$(find prl_ur5_description)/config/${setup_file['fixed_cameras_file']}"/>
     </xacro:if>
     <!-- back wall -->

Commit message: WiP: Small dimension adjustments

File: prl_ur5_description/urdf/_fixed_cameras.urdf.xacro (robot description, xacro)
@@ -43,6 +43,6 @@
         <xacro:property name="extrusion_width" value="${0.045 +0.02}"/> <!-- +/-1cm margin on the real size -->
         <xacro:property name="hr_z_pos" value="-0.05625"/> <!-- height at which the horizontal extrusion are fixed to the table -->
-        <xacro:property name="sj_height" value="${0.17 + 0.09}"/> <!-- Height of the spherical joint supporting the camera (plus the supporting part under) -->
-        <xacro:property name="sj_diameter" value="${0.045 +0.02}"/> <!-- Diameter of the spherical joint supporting the camera (plus the supporting part under) -->
+        <xacro:property name="sj_height" value="${0.08 + 0.09}"/> <!-- Height of the spherical joint supporting the camera + the angle piece supporting the spherical joint -->
+        <xacro:property name="sj_diameter" value="${0.09 +0.015}"/> <!-- Diameter of the spherical joint supporting the camera -->
         <!-- Simple math to change the side of the table to which the fixture is attached-->
         <xacro:if value="${camera['fixture_orientation'] == '+x'}">
@@ -70,5 +70,5 @@
             <xacro:property name="hr_z_rot" value="-1.570796327"/>
         </xacro:if>
-        <xacro:property name="vt_len" value="${camera['pose']['z'] - camera['offset']['z'] - hr_z_pos + extrusion_width}"/>
+        <xacro:property name="vt_len" value="${camera['pose']['z'] - camera['offset']['z'] - camera['size']['z']/2. - hr_z_pos + extrusion_width}"/>
         <!-- Horizontal extrusion -->
         <link name="hr_${camera['name']}">
@@ -111,5 +111,5 @@
             <parent link = "${parent}"/>
             <child link="vt_${camera['name']}"/>
-            <origin xyz="${camera['pose']['x'] - camera['offset']['x']} ${camera['pose']['y'] - camera['offset']['y']} ${camera['pose']['z']-camera['offset']['z']-vt_len/2.}" rpy="0 0 0"/>
+            <origin xyz="${camera['pose']['x'] - camera['offset']['x']} ${camera['pose']['y'] - camera['offset']['y']} ${vt_len/2. + hr_z_pos - extrusion_width}" rpy="0 0 0"/>
         </joint>
         <!-- Spherical joint holding the camera -->
@@ -132,5 +132,5 @@
             <parent link = "${parent}"/>
             <child link="sj_${camera['name']}"/>
-            <origin xyz="${camera['pose']['x']} ${camera['pose']['y']} ${camera['pose']['z'] - sj_height/2.}" rpy="0 0 0"/>
+            <origin xyz="${camera['pose']['x']} ${camera['pose']['y']} ${camera['pose']['z'] - camera['size']['z']/2. - sj_height/2.}" rpy="0 0 0"/>
         </joint>
     </xacro:macro>

Commit message: WiP: Color adjustment

File: prl_ur5_description/urdf/_fixed_cameras.urdf.xacro (robot description, xacro)
@@ -24,5 +24,5 @@
                     <box size="${camera['size']['x']} ${camera['size']['y']} ${camera['size']['z']}" />
                 </geometry>
-                <material name="purple"><color rgba="0.8 0 0.8 1"/></material>
+                <material name="purple"><color rgba="0.01 0.32 0.41 1"/></material>
             </visual>
             <collision>
@@ -77,4 +77,5 @@
                     <box size="${hr_len} ${extrusion_width} ${extrusion_width}" />
                 </geometry>
+                <material name="purple"/>
             </visual>
             <collision>
@@ -98,4 +99,5 @@
                     <box size="${extrusion_width} ${extrusion_width} ${vt_len}" />
                 </geometry>
+                <material name="purple"/>
             </visual>
             <collision>
@@ -119,4 +121,5 @@
                     <cylinder radius="${sj_diameter/2}" length="${sj_height}"/>
                 </geometry>
+                <material name="purple"/>
             </visual>
             <collision>

Commit message: WiP: update srdf

File: prl_ur5_description/urdf/_fixed_cameras.urdf.xacro (robot description, xacro)
@@ -4,20 +4,20 @@
     <xacro:macro name="fixed_cameras" params="parent fixed_cameras_file">
         <xacro:property name="fixed_cameras" value="${load_yaml(fixed_cameras_file)}"/>
-        <xacro:fixed_cameras_loop parent="${parent}" cameras="${fixed_cameras}"/>
+        <xacro:fixed_cameras_loop parent="${parent}" number="0" cameras="${fixed_cameras}"/>
     </xacro:macro>
     <!-- Reccursive macro to iterate over all the cameras -->
-    <xacro:macro name="fixed_cameras_loop" params="parent cameras">
+    <xacro:macro name="fixed_cameras_loop" params="parent number cameras">
         <xacro:if value="${cameras}">
                 <!-- pop first item from list -->
                 <xacro:property name="camera" value="${cameras.pop(0)}"/>
-                <xacro:fixed_camera parent="${parent}" camera="${camera}"/>
+                <xacro:fixed_camera parent="${parent}" number="${number}" camera="${camera}"/>
                 <!-- recursively call myself -->
-                <xacro:fixed_cameras_loop parent="${parent}" cameras="${cameras}"/>
+                <xacro:fixed_cameras_loop parent="${parent}" number="${number+1}" cameras="${cameras}"/>
         </xacro:if>
     </xacro:macro>
     <!-- Build one camera with its stand -->
-    <xacro:macro name="fixed_camera" params="parent camera">
+    <xacro:macro name="fixed_camera" params="parent number camera">
         <!-- Camera -->
-        <link name="camera_${camera['name']}">
+        <link name="fixed_camera_${number}">
             <visual>
                 <geometry>
@@ -32,10 +32,10 @@
             </collision>
         </link>
-        <gazebo reference="camera_${camera['name']}">
+        <gazebo reference="fixed_camera_${number}">
                 <material>Gazebo/BlueGlow</material>
         </gazebo>
-        <joint name="camera_${camera['name']}_fix" type="fixed">
+        <joint name="fixed_camera_${number}_fix" type="fixed">
             <parent link = "${parent}"/>
-            <child link="camera_${camera['name']}"/>
+            <child link="fixed_camera_${number}"/>
             <origin xyz="${camera['pose']['x']} ${camera['pose']['y']} ${camera['pose']['z']}" rpy="${camera['pose']['roll']} ${camera['pose']['pitch']} ${camera['pose']['yaw']}"/>
         </joint>
@@ -72,5 +72,5 @@
         <xacro:property name="vt_len" value="${camera['pose']['z'] - camera['offset']['z'] - camera['size']['z']/2. - hr_z_pos + extrusion_width}"/>
         <!-- Horizontal extrusion -->
-        <link name="hr_${camera['name']}">
+        <link name="fixed_hr_${number}">
             <visual>
                 <geometry>
@@ -85,14 +85,14 @@
             </collision>
         </link>
-        <gazebo reference="hr_${camera['name']}">
+        <gazebo reference="fixed_hr_${number}">
                 <material>Gazebo/BlueGlow</material>
         </gazebo>
-        <joint name="hr_${camera['name']}_fix" type="fixed">
+        <joint name="fixed_hr_${number}_fix" type="fixed">
             <parent link = "${parent}"/>
-            <child link="hr_${camera['name']}"/>
+            <child link="fixed_hr_${number}"/>
             <origin xyz="${hr_x_pos} ${hr_y_pos} ${hr_z_pos - extrusion_width/2.}" rpy="0 0 ${hr_z_rot}"/>
         </joint>
         <!-- Vertical extrusion -->
-        <link name="vt_${camera['name']}">
+        <link name="fixed_vt_${number}">
             <visual>
                 <geometry>
@@ -107,14 +107,14 @@
             </collision>
         </link>
-        <gazebo reference="vt_${camera['name']}">
+        <gazebo reference="fixed_vt_${number}">
                 <material>Gazebo/BlueGlow</material>
         </gazebo>
-        <joint name="vt_${camera['name']}_fix" type="fixed">
+        <joint name="fixed_vt_${number}_fix" type="fixed">
             <parent link = "${parent}"/>
-            <child link="vt_${camera['name']}"/>
+            <child link="fixed_vt_${number}"/>
             <origin xyz="${camera['pose']['x'] - camera['offset']['x']} ${camera['pose']['y'] - camera['offset']['y']} ${vt_len/2. + hr_z_pos - extrusion_width}" rpy="0 0 0"/>
         </joint>
         <!-- Spherical joint holding the camera -->
-        <link name="sj_${camera['name']}">
+        <link name="fixed_sj_${number}">
             <visual>
                 <geometry>
@@ -129,10 +129,10 @@
             </collision>
         </link>
-        <gazebo reference="sj_${camera['name']}">
+        <gazebo reference="fixed_sj_${number}">
                 <material>Gazebo/BlueGlow</material>
         </gazebo>
-        <joint name="sj_${camera['name']}_fix" type="fixed">
+        <joint name="fixed_sj_${number}_fix" type="fixed">
             <parent link = "${parent}"/>
-            <child link="sj_${camera['name']}"/>
+            <child link="fixed_sj_${number}"/>
             <origin xyz="${camera['pose']['x']} ${camera['pose']['y']} ${camera['pose']['z'] - camera['size']['z']/2. - sj_height/2.}" rpy="0 0 0"/>
         </joint>

Commit message: Disable fixture autocollision

File: prl_ur5_description/urdf/_fixed_cameras.urdf.xacro (robot description, xacro)
@@ -48,5 +48,5 @@
         <xacro:if value="${camera['fixture_orientation'] == '+x'}">
             <xacro:property name="hr_len" value="${camera['pose']['x'] - camera['offset']['x']}"/>
-            <xacro:property name="hr_x_pos" value="${hr_len/2.}"/>
+            <xacro:property name="hr_x_pos" value="${hr_len/2. + extrusion_width/2}"/>
             <xacro:property name="hr_y_pos" value="${camera['pose']['y'] - camera['offset']['y']}"/>
             <xacro:property name="hr_z_rot" value="0"/>
@@ -54,5 +54,5 @@
         <xacro:if value="${camera['fixture_orientation'] == '-x'}">
             <xacro:property name="hr_len" value="${-camera['pose']['x'] + camera['offset']['x']}"/>
-            <xacro:property name="hr_x_pos" value="${-hr_len/2.}"/>
+            <xacro:property name="hr_x_pos" value="${-hr_len/2. - extrusion_width/2.}"/>
             <xacro:property name="hr_y_pos" value="${camera['pose']['y'] - camera['offset']['y']}"/>
             <xacro:property name="hr_z_rot" value="3.1415926"/>
@@ -61,5 +61,5 @@
             <xacro:property name="hr_len" value="${camera['pose']['y'] - camera['offset']['y']}"/>
             <xacro:property name="hr_x_pos" value="${camera['pose']['x'] - camera['offset']['x']}"/>
-            <xacro:property name="hr_y_pos" value="${hr_len/2.}"/>
+            <xacro:property name="hr_y_pos" value="${hr_len/2. + extrusion_width/2.}"/>
             <xacro:property name="hr_z_rot" value="1.570796327"/>
         </xacro:if>
@@ -67,8 +67,8 @@
             <xacro:property name="hr_len" value="${-camera['pose']['y'] + camera['offset']['y']}"/>
             <xacro:property name="hr_x_pos" value="${camera['pose']['x'] - camera['offset']['x']}"/>
-            <xacro:property name="hr_y_pos" value="${-hr_len/2.}"/>
+            <xacro:property name="hr_y_pos" value="${-hr_len/2. - extrusion_width/2.}"/>
             <xacro:property name="hr_z_rot" value="-1.570796327"/>
         </xacro:if>
-        <xacro:property name="vt_len" value="${camera['pose']['z'] - camera['offset']['z'] - camera['size']['z']/2. - hr_z_pos + extrusion_width}"/>
+        <xacro:property name="vt_len" value="${camera['pose']['z'] - camera['offset']['z'] - camera['size']['z']/2. - hr_z_pos}"/>
         <!-- Horizontal extrusion -->
         <link name="fixed_hr_${number}">
@@ -113,5 +113,5 @@
             <parent link = "${parent}"/>
             <child link="fixed_vt_${number}"/>
-            <origin xyz="${camera['pose']['x'] - camera['offset']['x']} ${camera['pose']['y'] - camera['offset']['y']} ${vt_len/2. + hr_z_pos - extrusion_width}" rpy="0 0 0"/>
+            <origin xyz="${camera['pose']['x'] - camera['offset']['x']} ${camera['pose']['y'] - camera['offset']['y']} ${vt_len/2. + hr_z_pos}" rpy="0 0 0"/>
         </joint>
         <!-- Spherical joint holding the camera -->

Commit message: Fixture are not touching the table anymore

File: prl_ur5_description/urdf/_fixed_cameras.urdf.xacro (robot description, xacro)
@@ -46,26 +46,27 @@
         <xacro:property name="sj_diameter" value="${0.09 +0.015}"/> <!-- Diameter of the spherical joint supporting the camera -->
         <!-- Simple math to change the side of the table to which the fixture is attached-->
+        <!-- The arbitrary values 0.92 0.92 0.29 0.52 correspond to the dimensions of the table with 1cm margin, so the extrusions are not touching the table-->
         <xacro:if value="${camera['fixture_orientation'] == '+x'}">
-            <xacro:property name="hr_len" value="${camera['pose']['x'] - camera['offset']['x']}"/>
-            <xacro:property name="hr_x_pos" value="${hr_len/2. + extrusion_width/2}"/>
+            <xacro:property name="hr_len" value="${camera['pose']['x'] - camera['offset']['x'] + extrusion_width/2. - 0.92}"/>
+            <xacro:property name="hr_x_pos" value="${hr_len/2. + 0.92}"/>
             <xacro:property name="hr_y_pos" value="${camera['pose']['y'] - camera['offset']['y']}"/>
             <xacro:property name="hr_z_rot" value="0"/>
         </xacro:if>
         <xacro:if value="${camera['fixture_orientation'] == '-x'}">
-            <xacro:property name="hr_len" value="${-camera['pose']['x'] + camera['offset']['x']}"/>
-            <xacro:property name="hr_x_pos" value="${-hr_len/2. - extrusion_width/2.}"/>
+            <xacro:property name="hr_len" value="${-camera['pose']['x'] + camera['offset']['x'] + extrusion_width/2. - 0.92}"/>
+            <xacro:property name="hr_x_pos" value="${-hr_len/2. - 0.92}"/>
             <xacro:property name="hr_y_pos" value="${camera['pose']['y'] - camera['offset']['y']}"/>
             <xacro:property name="hr_z_rot" value="3.1415926"/>
         </xacro:if>
         <xacro:if value="${camera['fixture_orientation'] == '+y'}">
-            <xacro:property name="hr_len" value="${camera['pose']['y'] - camera['offset']['y']}"/>
+            <xacro:property name="hr_len" value="${camera['pose']['y'] - camera['offset']['y'] + extrusion_width/2.  - 0.29}"/>
             <xacro:property name="hr_x_pos" value="${camera['pose']['x'] - camera['offset']['x']}"/>
-            <xacro:property name="hr_y_pos" value="${hr_len/2. + extrusion_width/2.}"/>
+            <xacro:property name="hr_y_pos" value="${hr_len/2. + 0.29}"/>
             <xacro:property name="hr_z_rot" value="1.570796327"/>
         </xacro:if>
         <xacro:if value="${camera['fixture_orientation'] == '-y'}">
-            <xacro:property name="hr_len" value="${-camera['pose']['y'] + camera['offset']['y']}"/>
+            <xacro:property name="hr_len" value="${-camera['pose']['y'] + camera['offset']['y'] + extrusion_width/2.  - 0.52}"/>
             <xacro:property name="hr_x_pos" value="${camera['pose']['x'] - camera['offset']['x']}"/>
-            <xacro:property name="hr_y_pos" value="${-hr_len/2. - extrusion_width/2.}"/>
+            <xacro:property name="hr_y_pos" value="${-hr_len/2. - 0.52}"/>
             <xacro:property name="hr_z_rot" value="-1.570796327"/>
         </xacro:if>
