Commit message: Proper fixture link chain for preventing self collision (without srdf)

File: prl_ur5_description/urdf/_fixed_cameras.urdf.xacro (robot description, xacro)
@@ -42,5 +42,5 @@
         <!-- Numerical dimensions for the fixtures -->
         <xacro:property name="extrusion_width" value="${0.045 +0.02}"/> <!-- +/-1cm margin on the real size -->
-        <xacro:property name="hr_z_pos" value="-0.05625"/> <!-- height at which the horizontal extrusion are fixed to the table -->
+        <xacro:property name="hr_z_pos_absolute" value="-0.05625"/> <!-- height at which the horizontal extrusion are fixed to the table -->
         <xacro:property name="sj_height" value="${0.08 + 0.09}"/> <!-- Height of the spherical joint supporting the camera + the angle piece supporting the spherical joint -->
         <xacro:property name="sj_diameter" value="${0.09 +0.015}"/> <!-- Diameter of the spherical joint supporting the camera -->
@@ -49,32 +49,32 @@
         <xacro:if value="${camera['fixture_orientation'] == '+x'}">
             <xacro:property name="hr_len" value="${camera['pose']['x'] - camera['offset']['x'] + extrusion_width/2. - 0.92}"/>
-            <xacro:property name="hr_x_pos" value="${hr_len/2. + 0.92}"/>
-            <xacro:property name="hr_y_pos" value="${camera['pose']['y'] - camera['offset']['y']}"/>
-            <xacro:property name="hr_z_rot" value="0"/>
+            <xacro:property name="hr_x_pos_relative" value="${- hr_len/2. + extrusion_width/2.}"/>
+            <xacro:property name="hr_y_pos_relative" value="0"/>
+            <xacro:property name="hr_z_rot_relative" value="0"/>
         </xacro:if>
         <xacro:if value="${camera['fixture_orientation'] == '-x'}">
             <xacro:property name="hr_len" value="${-camera['pose']['x'] + camera['offset']['x'] + extrusion_width/2. - 0.92}"/>
-            <xacro:property name="hr_x_pos" value="${-hr_len/2. - 0.92}"/>
-            <xacro:property name="hr_y_pos" value="${camera['pose']['y'] - camera['offset']['y']}"/>
-            <xacro:property name="hr_z_rot" value="3.1415926"/>
+            <xacro:property name="hr_x_pos_relative" value="${hr_len/2. - extrusion_width/2.}"/>
+            <xacro:property name="hr_y_pos_relative" value="0"/>
+            <xacro:property name="hr_z_rot_relative" value="3.1415926"/>
         </xacro:if>
         <xacro:if value="${camera['fixture_orientation'] == '+y'}">
             <xacro:property name="hr_len" value="${camera['pose']['y'] - camera['offset']['y'] + extrusion_width/2.  - 0.29}"/>
-            <xacro:property name="hr_x_pos" value="${camera['pose']['x'] - camera['offset']['x']}"/>
-            <xacro:property name="hr_y_pos" value="${hr_len/2. + 0.29}"/>
-            <xacro:property name="hr_z_rot" value="1.570796327"/>
+            <xacro:property name="hr_x_pos_relative" value="0"/>
+            <xacro:property name="hr_y_pos_relative" value="${- hr_len/2. + extrusion_width/2.}"/>
+            <xacro:property name="hr_z_rot_relative" value="1.570796327"/>
         </xacro:if>
         <xacro:if value="${camera['fixture_orientation'] == '-y'}">
             <xacro:property name="hr_len" value="${-camera['pose']['y'] + camera['offset']['y'] + extrusion_width/2.  - 0.52}"/>
-            <xacro:property name="hr_x_pos" value="${camera['pose']['x'] - camera['offset']['x']}"/>
-            <xacro:property name="hr_y_pos" value="${-hr_len/2. - 0.52}"/>
-            <xacro:property name="hr_z_rot" value="-1.570796327"/>
+            <xacro:property name="hr_x_pos_relative" value="0"/>
+            <xacro:property name="hr_y_pos_relative" value="${hr_len/2. - extrusion_width/2.}"/>
+            <xacro:property name="hr_z_rot_relative" value="-1.570796327"/>
         </xacro:if>
-        <xacro:property name="vt_len" value="${camera['pose']['z'] - camera['offset']['z'] - camera['size']['z']/2. - hr_z_pos}"/>
-        <!-- Horizontal extrusion -->
-        <link name="fixed_hr_${number}">
+        <xacro:property name="vt_len" value="${camera['pose']['z'] - camera['offset']['z'] - hr_z_pos_absolute}"/>
+        <!-- Spherical joint holding the camera -->
+        <link name="fixed_sj_${number}">
             <visual>
                 <geometry>
-                    <box size="${hr_len} ${extrusion_width} ${extrusion_width}" />
+                    <cylinder radius="${sj_diameter/2}" length="${sj_height}"/>
                 </geometry>
                 <material name="purple"/>
@@ -82,15 +82,15 @@
             <collision>
                 <geometry>
-                    <box size="${hr_len} ${extrusion_width} ${extrusion_width}" />
+                    <cylinder radius="${sj_diameter/2}" length="${sj_height}"/>
                 </geometry>
             </collision>
         </link>
-        <gazebo reference="fixed_hr_${number}">
+        <gazebo reference="fixed_sj_${number}">
                 <material>Gazebo/BlueGlow</material>
         </gazebo>
-        <joint name="fixed_hr_${number}_fix" type="fixed">
-            <parent link = "${parent}"/>
-            <child link="fixed_hr_${number}"/>
-            <origin xyz="${hr_x_pos} ${hr_y_pos} ${hr_z_pos - extrusion_width/2.}" rpy="0 0 ${hr_z_rot}"/>
+        <joint name="fixed_sj_${number}_fix" type="fixed">
+            <parent link = "fixed_camera_${number}"/>
+            <child link="fixed_sj_${number}"/>
+            <origin xyz="0 0 ${- camera['size']['z']/2. - sj_height/2.}" rpy="${-camera['pose']['roll']} ${-camera['pose']['pitch']} ${-camera['pose']['yaw']}"/>
         </joint>
         <!-- Vertical extrusion -->
@@ -112,13 +112,13 @@
         </gazebo>
         <joint name="fixed_vt_${number}_fix" type="fixed">
-            <parent link = "${parent}"/>
+            <parent link = "fixed_sj_${number}"/>
             <child link="fixed_vt_${number}"/>
-            <origin xyz="${camera['pose']['x'] - camera['offset']['x']} ${camera['pose']['y'] - camera['offset']['y']} ${vt_len/2. + hr_z_pos}" rpy="0 0 0"/>
+            <origin xyz="${-camera['offset']['x']} ${-camera['offset']['y']} ${sj_height/2. + camera['size']['z']/2. - camera['offset']['z'] - vt_len/2.}" rpy="0 0 0"/>
         </joint>
-        <!-- Spherical joint holding the camera -->
-        <link name="fixed_sj_${number}">
+        <!-- Horizontal extrusion -->
+        <link name="fixed_hr_${number}">
             <visual>
                 <geometry>
-                    <cylinder radius="${sj_diameter/2}" length="${sj_height}"/>
+                    <box size="${hr_len} ${extrusion_width} ${extrusion_width}" />
                 </geometry>
                 <material name="purple"/>
@@ -126,15 +126,15 @@
             <collision>
                 <geometry>
-                    <cylinder radius="${sj_diameter/2}" length="${sj_height}"/>
+                    <box size="${hr_len} ${extrusion_width} ${extrusion_width}" />
                 </geometry>
             </collision>
         </link>
-        <gazebo reference="fixed_sj_${number}">
+        <gazebo reference="fixed_hr_${number}">
                 <material>Gazebo/BlueGlow</material>
         </gazebo>
-        <joint name="fixed_sj_${number}_fix" type="fixed">
-            <parent link = "${parent}"/>
-            <child link="fixed_sj_${number}"/>
-            <origin xyz="${camera['pose']['x']} ${camera['pose']['y']} ${camera['pose']['z'] - camera['size']['z']/2. - sj_height/2.}" rpy="0 0 0"/>
+        <joint name="fixed_hr_${number}_fix" type="fixed">
+            <parent link = "fixed_vt_${number}"/>
+            <child link="fixed_hr_${number}"/>
+            <origin xyz="${hr_x_pos_relative} ${hr_y_pos_relative} ${- vt_len/2. - extrusion_width/2.}" rpy="0 0 ${hr_z_rot_relative}"/>
         </joint>
     </xacro:macro>

Commit message: Simplify model : remove camera orientation and model it as a cylinder

File: prl_ur5_description/urdf/_fixed_cameras.urdf.xacro (robot description, xacro)
@@ -18,9 +18,41 @@
     <!-- Build one camera with its stand -->
     <xacro:macro name="fixed_camera" params="parent number camera">
+        <!-- Numerical dimensions for the fixtures -->
+        <xacro:property name="extrusion_width" value="${0.045 +0.02}"/> <!-- +/-1cm margin on the real size -->
+        <xacro:property name="hr_z_pos_absolute" value="-0.05625"/> <!-- height at which the horizontal extrusion are fixed to the table -->
+        <xacro:property name="sj_height" value="${0.08 + 0.09}"/> <!-- Height of the spherical joint supporting the camera + the angle piece supporting the spherical joint -->
+        <xacro:property name="sj_diameter" value="${0.09 +0.015}"/> <!-- Diameter of the spherical joint supporting the camera -->
+        <!-- Simple math to change the side of the table to which the fixture is attached-->
+        <!-- The arbitrary values 0.92 0.92 0.29 0.52 correspond to the dimensions of the table with 1cm margin, so the extrusions are not touching the table-->
+        <xacro:if value="${camera['fixture_orientation'] == '+x'}">
+            <xacro:property name="hr_len" value="${camera['position']['x'] - camera['offset']['x'] + extrusion_width/2. - 0.92}"/>
+            <xacro:property name="hr_x_pos_relative" value="${- hr_len/2. + extrusion_width/2.}"/>
+            <xacro:property name="hr_y_pos_relative" value="0"/>
+            <xacro:property name="hr_z_rot_relative" value="0"/>
+        </xacro:if>
+        <xacro:if value="${camera['fixture_orientation'] == '-x'}">
+            <xacro:property name="hr_len" value="${-camera['position']['x'] + camera['offset']['x'] + extrusion_width/2. - 0.92}"/>
+            <xacro:property name="hr_x_pos_relative" value="${hr_len/2. - extrusion_width/2.}"/>
+            <xacro:property name="hr_y_pos_relative" value="0"/>
+            <xacro:property name="hr_z_rot_relative" value="3.1415926"/>
+        </xacro:if>
+        <xacro:if value="${camera['fixture_orientation'] == '+y'}">
+            <xacro:property name="hr_len" value="${camera['position']['y'] - camera['offset']['y'] + extrusion_width/2.  - 0.29}"/>
+            <xacro:property name="hr_x_pos_relative" value="0"/>
+            <xacro:property name="hr_y_pos_relative" value="${- hr_len/2. + extrusion_width/2.}"/>
+            <xacro:property name="hr_z_rot_relative" value="1.570796327"/>
+        </xacro:if>
+        <xacro:if value="${camera['fixture_orientation'] == '-y'}">
+            <xacro:property name="hr_len" value="${-camera['position']['y'] + camera['offset']['y'] + extrusion_width/2.  - 0.52}"/>
+            <xacro:property name="hr_x_pos_relative" value="0"/>
+            <xacro:property name="hr_y_pos_relative" value="${hr_len/2. - extrusion_width/2.}"/>
+            <xacro:property name="hr_z_rot_relative" value="-1.570796327"/>
+        </xacro:if>
+        <xacro:property name="vt_len" value="${camera['position']['z'] - camera['offset']['z'] - hr_z_pos_absolute}"/>
         <!-- Camera -->
         <link name="fixed_camera_${number}">
             <visual>
                 <geometry>
-                    <box size="${camera['size']['x']} ${camera['size']['y']} ${camera['size']['z']}" />
+                    <cylinder radius="${camera['size']['width']/2.}" length="${camera['size']['height']}"/>
                 </geometry>
                 <material name="purple"><color rgba="0.01 0.32 0.41 1"/></material>
@@ -28,5 +60,5 @@
             <collision>
                 <geometry>
-                    <box size="${camera['size']['x']} ${camera['size']['y']} ${camera['size']['z']}" />
+                    <cylinder radius="${camera['size']['width']/2.}" length="${camera['size']['height']}"/>
                 </geometry>
             </collision>
@@ -38,38 +70,6 @@
             <parent link = "${parent}"/>
             <child link="fixed_camera_${number}"/>
-            <origin xyz="${camera['pose']['x']} ${camera['pose']['y']} ${camera['pose']['z']}" rpy="${camera['pose']['roll']} ${camera['pose']['pitch']} ${camera['pose']['yaw']}"/>
+            <origin xyz="${camera['position']['x']} ${camera['position']['y']} ${camera['position']['z']}" rpy="0 0 0"/>
         </joint>
-        <!-- Numerical dimensions for the fixtures -->
-        <xacro:property name="extrusion_width" value="${0.045 +0.02}"/> <!-- +/-1cm margin on the real size -->
-        <xacro:property name="hr_z_pos_absolute" value="-0.05625"/> <!-- height at which the horizontal extrusion are fixed to the table -->
-        <xacro:property name="sj_height" value="${0.08 + 0.09}"/> <!-- Height of the spherical joint supporting the camera + the angle piece supporting the spherical joint -->
-        <xacro:property name="sj_diameter" value="${0.09 +0.015}"/> <!-- Diameter of the spherical joint supporting the camera -->
-        <!-- Simple math to change the side of the table to which the fixture is attached-->
-        <!-- The arbitrary values 0.92 0.92 0.29 0.52 correspond to the dimensions of the table with 1cm margin, so the extrusions are not touching the table-->
-        <xacro:if value="${camera['fixture_orientation'] == '+x'}">
-            <xacro:property name="hr_len" value="${camera['pose']['x'] - camera['offset']['x'] + extrusion_width/2. - 0.92}"/>
-            <xacro:property name="hr_x_pos_relative" value="${- hr_len/2. + extrusion_width/2.}"/>
-            <xacro:property name="hr_y_pos_relative" value="0"/>
-            <xacro:property name="hr_z_rot_relative" value="0"/>
-        </xacro:if>
-        <xacro:if value="${camera['fixture_orientation'] == '-x'}">
-            <xacro:property name="hr_len" value="${-camera['pose']['x'] + camera['offset']['x'] + extrusion_width/2. - 0.92}"/>
-            <xacro:property name="hr_x_pos_relative" value="${hr_len/2. - extrusion_width/2.}"/>
-            <xacro:property name="hr_y_pos_relative" value="0"/>
-            <xacro:property name="hr_z_rot_relative" value="3.1415926"/>
-        </xacro:if>
-        <xacro:if value="${camera['fixture_orientation'] == '+y'}">
-            <xacro:property name="hr_len" value="${camera['pose']['y'] - camera['offset']['y'] + extrusion_width/2.  - 0.29}"/>
-            <xacro:property name="hr_x_pos_relative" value="0"/>
-            <xacro:property name="hr_y_pos_relative" value="${- hr_len/2. + extrusion_width/2.}"/>
-            <xacro:property name="hr_z_rot_relative" value="1.570796327"/>
-        </xacro:if>
-        <xacro:if value="${camera['fixture_orientation'] == '-y'}">
-            <xacro:property name="hr_len" value="${-camera['pose']['y'] + camera['offset']['y'] + extrusion_width/2.  - 0.52}"/>
-            <xacro:property name="hr_x_pos_relative" value="0"/>
-            <xacro:property name="hr_y_pos_relative" value="${hr_len/2. - extrusion_width/2.}"/>
-            <xacro:property name="hr_z_rot_relative" value="-1.570796327"/>
-        </xacro:if>
-        <xacro:property name="vt_len" value="${camera['pose']['z'] - camera['offset']['z'] - hr_z_pos_absolute}"/>
         <!-- Spherical joint holding the camera -->
         <link name="fixed_sj_${number}">
@@ -92,5 +92,5 @@
             <parent link = "fixed_camera_${number}"/>
             <child link="fixed_sj_${number}"/>
-            <origin xyz="0 0 ${- camera['size']['z']/2. - sj_height/2.}" rpy="${-camera['pose']['roll']} ${-camera['pose']['pitch']} ${-camera['pose']['yaw']}"/>
+            <origin xyz="0 0 ${- camera['size']['height']/2. - sj_height/2.}" rpy="0 0 0"/>
         </joint>
         <!-- Vertical extrusion -->
@@ -114,5 +114,5 @@
             <parent link = "fixed_sj_${number}"/>
             <child link="fixed_vt_${number}"/>
-            <origin xyz="${-camera['offset']['x']} ${-camera['offset']['y']} ${sj_height/2. + camera['size']['z']/2. - camera['offset']['z'] - vt_len/2.}" rpy="0 0 0"/>
+            <origin xyz="${-camera['offset']['x']} ${-camera['offset']['y']} ${sj_height/2. + camera['size']['height']/2. - camera['offset']['z'] - vt_len/2.}" rpy="0 0 0"/>
         </joint>
         <!-- Horizontal extrusion -->

Commit message: Raise camera support margin

File: prl_ur5_description/urdf/_fixed_cameras.urdf.xacro (robot description, xacro)
@@ -19,5 +19,5 @@
     <xacro:macro name="fixed_camera" params="parent number camera">
         <!-- Numerical dimensions for the fixtures -->
-        <xacro:property name="extrusion_width" value="${0.045 +0.02}"/> <!-- +/-1cm margin on the real size -->
+        <xacro:property name="extrusion_width" value="${0.045 +0.04}"/> <!-- +/-2cm margin on the real size -->
         <xacro:property name="hr_z_pos_absolute" value="-0.05625"/> <!-- height at which the horizontal extrusion are fixed to the table -->
         <xacro:property name="sj_height" value="${0.08 + 0.09}"/> <!-- Height of the spherical joint supporting the camera + the angle piece supporting the spherical joint -->

Commit message: Increase external cameras safety margin

File: prl_ur5_description/urdf/_fixed_cameras.urdf.xacro (robot description, xacro)
@@ -19,8 +19,8 @@
     <xacro:macro name="fixed_camera" params="parent number camera">
         <!-- Numerical dimensions for the fixtures -->
-        <xacro:property name="extrusion_width" value="${0.045 +0.04}"/> <!-- +/-2cm margin on the real size -->
+        <xacro:property name="extrusion_width" value="${0.045 +0.06}"/> <!-- +/-3cm margin on the real size -->
         <xacro:property name="hr_z_pos_absolute" value="-0.05625"/> <!-- height at which the horizontal extrusion are fixed to the table -->
         <xacro:property name="sj_height" value="${0.08 + 0.09}"/> <!-- Height of the spherical joint supporting the camera + the angle piece supporting the spherical joint -->
-        <xacro:property name="sj_diameter" value="${0.09 +0.015}"/> <!-- Diameter of the spherical joint supporting the camera -->
+        <xacro:property name="sj_diameter" value="${0.09 +0.03}"/> <!-- Diameter of the spherical joint supporting the camera -->
         <!-- Simple math to change the side of the table to which the fixture is attached-->
         <!-- The arbitrary values 0.92 0.92 0.29 0.52 correspond to the dimensions of the table with 1cm margin, so the extrusions are not touching the table-->

Commit message: Fixing deprecation warnings

File: prl_ur5_description/urdf/_fixed_cameras.urdf.xacro (robot description, xacro)
@@ -3,5 +3,5 @@
     <!-- Build fixed camera with their support from one file -->
     <xacro:macro name="fixed_cameras" params="parent fixed_cameras_file">
-        <xacro:property name="fixed_cameras" value="${load_yaml(fixed_cameras_file)}"/>
+        <xacro:property name="fixed_cameras" value="${xacro.load_yaml(fixed_cameras_file)}"/>
         <xacro:fixed_cameras_loop parent="${parent}" number="0" cameras="${fixed_cameras}"/>
     </xacro:macro>

File: prl_ur5_description/urdf/prl_ur5_robot.urdf.xacro (robot description, xacro)
@@ -7,5 +7,5 @@
   <!-- ur5 robot -->
   <xacro:include filename="$(find prl_ur5_description)/urdf/prl_ur5.urdf.xacro"/>
-  <xacro:prl_ur5 setup_file="${load_yaml('$(find prl_ur5_robot_configuration)/config/$(arg setup).yaml')}"
+  <xacro:prl_ur5 setup_file="${xacro.load_yaml('$(find prl_ur5_robot_configuration)/config/$(arg setup).yaml')}"
                  table="$(arg table)"
                  hardware_interface="$(arg hardware_interface)"/>

Commit message: Replace xacro.load_yaml with load_yaml. Will create warnings in some cases but prevent crash for older xacro version (on conda)

File: prl_ur5_description/urdf/_fixed_cameras.urdf.xacro (robot description, xacro)
@@ -6,5 +6,5 @@
     <!-- Build fixed camera with their support from one file -->
     <xacro:macro name="fixed_cameras" params="parent fixed_cameras_file turn_on:=false">
-        <xacro:property name="fixed_cameras" value="${xacro.load_yaml(fixed_cameras_file)}"/>
+        <xacro:property name="fixed_cameras" value="${load_yaml(fixed_cameras_file)}"/>
         <xacro:fixed_cameras_loop parent="${parent}" number="0" cameras="${fixed_cameras}" turn_on="${turn_on}"/>
     </xacro:macro>

File: prl_ur5_description/urdf/prl_ur5_robot.urdf.xacro (robot description, xacro)
@@ -9,5 +9,5 @@
   <!-- ur5 robot -->
   <xacro:include filename="$(find prl_ur5_description)/urdf/prl_ur5.urdf.xacro"/>
-  <xacro:prl_ur5 setup_file="${xacro.load_yaml('$(find prl_ur5_robot_configuration)/config/$(arg setup).yaml')}"
+  <xacro:prl_ur5 setup_file="${load_yaml('$(find prl_ur5_robot_configuration)/config/$(arg setup).yaml')}"
                  table="$(arg table)"
                  hardware_interface="$(arg hardware_interface)"

File: prl_ur5_moveit_config/config/standart_setup/prl_ur5_robot.srdf.xacro (robot description, xacro)
@@ -6,5 +6,5 @@
 <robot xmlns:xacro="http://wiki.ros.org/xacro" name="prl_ur5_robot">
     <xacro:arg name="setup_name" default=""/>
-    <xacro:property name="setup" value="${xacro.load_yaml('$(find prl_ur5_robot_configuration)/config/$(arg setup_name).yaml')}"/>
+    <xacro:property name="setup" value="${load_yaml('$(find prl_ur5_robot_configuration)/config/$(arg setup_name).yaml')}"/>
     <!--GROUPS: Representation of a set of joints and links. This can be useful for specifying DOF to plan for, defining arms, end effectors, etc-->
     <!--LINKS: When a link is specified, the parent joint of that link (if it exists) is automatically included-->
@@ -207,5 +207,5 @@
     <!-- Iterate voer all cameras using reccursive function-->
     <xacro:property name="fixed_cameras_file" value="$(find prl_ur5_robot_configuration)/config/${setup['fixed_cameras_file']}"/>
-    <xacro:property name="fixed_cameras" value="${xacro.load_yaml(fixed_cameras_file)}"/>
+    <xacro:property name="fixed_cameras" value="${load_yaml(fixed_cameras_file)}"/>
     <xacro:macro name="external_cameras_loop" params="cameras number">
         <xacro:if value="${cameras}">
