Commit message: Possibility to use custom grippers / Simplify SRDF by using xacro / Update one depency repo uri

File: prl_ur5_description/urdf/_gripper.urdf.xacro (robot description, xacro)
@@ -5,5 +5,5 @@
   <xacro:macro name="gripper" params="gripper prefix parent pose hardware_interface">
     <!-- check gripper type -->
-    <xacro:unless value="${gripper in [None, 'onrobot-rg2', 'onrobot-rg6']}">
+    <xacro:unless value="${gripper in [None, 'onrobot-rg2', 'onrobot-rg6'] or gripper.startswith('custom:')}">
       <xacro:unknown_gripper_type/>
     </xacro:unless>
@@ -20,4 +20,11 @@
       </xacro:onrobot_rg>
     </xacro:if>
+    <!-- if custom gripper -->
+    <xacro:if value="${gripper.startswith('custom:')}">
+      <xacro:include filename="$(find prl_ur5_robot_configuration)/urdf/${gripper[7:]}.urdf.xacro"/>
+        <xacro:call macro="${gripper[7:]}" prefix='${prefix}gripper' parent="${parent}" transmission_hw_interface="${hardware_interface}">
+        <origin xyz="${pose['x']} ${pose['y']} ${pose['z']}" rpy="${pose['roll']} ${pose['pitch']} ${pose['yaw']}"/>
+      </xacro:call>
+    </xacro:if>
   </xacro:macro>
 </robot>

Commit message: Add RG6-v2 gripper

File: prl_ur5_description/urdf/_gripper.urdf.xacro (robot description, xacro)
@@ -5,5 +5,5 @@
   <xacro:macro name="gripper" params="gripper prefix parent pose hardware_interface">
     <!-- check gripper type -->
-    <xacro:unless value="${gripper in [None, 'onrobot-rg2', 'onrobot-rg6'] or gripper.startswith('custom:')}">
+    <xacro:unless value="${gripper in [None, 'onrobot-rg2', 'onrobot-rg6', 'onrobot-rg6-v2'] or gripper.startswith('custom:')}">
       <xacro:unknown_gripper_type/>
     </xacro:unless>
@@ -20,4 +20,10 @@
       </xacro:onrobot_rg>
     </xacro:if>
+    <!-- if onrobot-rg6-v2 -->
+    <xacro:if value="${gripper == 'onrobot-rg6-v2'}">
+      <xacro:onrobot_rg prefix='${prefix}gripper' parent="${parent}" model="rg6_v2" safety_shield="true" transmission_hw_interface="${hardware_interface}">
+        <origin xyz="${pose['x']} ${pose['y']} ${pose['z']}" rpy="${pose['roll']} ${pose['pitch']} ${pose['yaw']}"/>
+      </xacro:onrobot_rg>
+    </xacro:if>
     <!-- if custom gripper -->
     <xacro:if value="${gripper.startswith('custom:')}">

File: prl_ur5_moveit_config/config/standart_setup/prl_ur5_robot.srdf.xacro (robot description, xacro)
@@ -22,4 +22,8 @@
         <xacro:property name="left_gripper_name" value="onrobot_rg6"/>
     </xacro:if>
+    <!-- if onrobot-rg6-v2 -->
+    <xacro:if value="${setup['left']['gripper'] == 'onrobot-rg6-v2'}">
+        <xacro:property name="left_gripper_name" value="onrobot_rg6_v2"/>
+    </xacro:if>
     <!-- if custom gripper -->
     <xacro:if value="${setup['left']['gripper'].startswith('custom:')}">
@@ -46,4 +50,8 @@
     <xacro:if value="${setup['right']['gripper'] == 'onrobot-rg6'}">
         <xacro:property name="right_gripper_name" value="onrobot_rg6"/>
+    </xacro:if>
+    <!-- if onrobot-rg6 -->
+    <xacro:if value="${setup['right']['gripper'] == 'onrobot-rg6-v2'}">
+        <xacro:property name="right_gripper_name" value="onrobot_rg6_v2"/>
     </xacro:if>
     <!-- if custom gripper -->

Commit message: Add AllegroHand in urdf/srdf -- SRDF group now define in gripper lib

File: prl_ur5_description/urdf/_gripper.urdf.xacro (robot description, xacro)
@@ -5,5 +5,5 @@
   <xacro:macro name="gripper" params="gripper prefix parent pose hardware_interface">
     <!-- check gripper type -->
-    <xacro:unless value="${gripper in [None, 'onrobot-rg2', 'onrobot-rg6', 'onrobot-rg6-v2'] or gripper.startswith('custom:')}">
+    <xacro:unless value="${gripper in [None, 'onrobot-rg2', 'onrobot-rg6', 'onrobot-rg6-v2'] or gripper.startswith('custom:') or gripper.startswith('allegro-hand:')}">
       <xacro:unknown_gripper_type/>
     </xacro:unless>
@@ -26,4 +26,11 @@
       </xacro:onrobot_rg>
     </xacro:if>
+    <!-- if allegro-hand -->
+    <xacro:if value="${gripper.startswith('allegro-hand:')}">
+      <xacro:include filename="$(find allegro_hand_description)/allegro_hand_description.urdf.xacro"/>
+      <xacro:allegro_hand chirality='${gripper[13:]}' prefix='${prefix}gripper' parent="${parent}" last_links_inertia_factor="${20 if gz_sim else 1.0}">
+        <origin xyz="${pose['x']} ${pose['y']} ${pose['z']}" rpy="${pose['roll']} ${pose['pitch']} ${pose['yaw']}"/>
+      </xacro:allegro_hand>
+    </xacro:if>
     <!-- if custom gripper -->
     <xacro:if value="${gripper.startswith('custom:')}">

File: prl_ur5_moveit_config/config/standart_setup/prl_ur5_robot.srdf.xacro (robot description, xacro)
@@ -26,4 +26,9 @@
         <xacro:property name="left_gripper_name" value="onrobot_rg6_v2"/>
     </xacro:if>
+    <!-- if allegro-hand -->
+    <xacro:if value="${setup['left']['gripper'].startswith('allegro-hand:')}">
+      <xacro:include filename="$(find allegro_hand_description)/allegro_hand_description.srdf.xacro"/>
+      <xacro:property name="left_gripper_name" value="allegro_hand"/>
+    </xacro:if>
     <!-- if custom gripper -->
     <xacro:if value="${setup['left']['gripper'].startswith('custom:')}">
@@ -31,8 +36,7 @@
         <xacro:property name="left_gripper_name" value="${setup['left']['gripper'][7:]}"/>
     </xacro:if>
-    <!-- Create the group, the autocolision and collision tags-->
-    <group name="left_gripper">
-            <xacro:call macro="${left_gripper_name}_group" prefix='left_gripper'/>
-        </group>
+    <!-- Define gripper group and define its states-->
+    <xacro:call macro="${left_gripper_name}_group_define" group_name="left_gripper" prefix='left_gripper'/>
+    <!-- Create autocolision and collision tags -->
     <xacro:call macro="${left_gripper_name}_autocol" prefix='left_gripper'/>
     <xacro:call macro="${left_gripper_name}_col_with" prefix='left_gripper' link='left_wrist_3_link'/>
@@ -55,4 +59,9 @@
         <xacro:property name="right_gripper_name" value="onrobot_rg6_v2"/>
     </xacro:if>
+    <!-- if allegro-hand -->
+    <xacro:if value="${setup['right']['gripper'].startswith('allegro-hand:')}">
+      <xacro:include filename="$(find allegro_hand_description)/allegro_hand_description.srdf.xacro"/>
+      <xacro:property name="right_gripper_name" value="allegro_hand"/>
+    </xacro:if>
     <!-- if custom gripper -->
     <xacro:if value="${setup['right']['gripper'].startswith('custom:')}">
@@ -60,8 +69,7 @@
         <xacro:property name="right_gripper_name" value="${setup['right']['gripper'][7:]}"/>
     </xacro:if>
-    <!-- Create the group, the autocolision and collision tags-->
-    <group name="right_gripper">
-        <xacro:call macro="${right_gripper_name}_group" prefix='right_gripper'/>
-    </group>
+    <!-- Define gripper group and define its states-->
+    <xacro:call macro="${right_gripper_name}_group_define" group_name='right_gripper' prefix='right_gripper'/>
+    <!-- Create autocolision and collision tags -->
     <xacro:call macro="${right_gripper_name}_autocol" prefix='right_gripper'/>
     <xacro:call macro="${right_gripper_name}_col_with" prefix='right_gripper' link='right_wrist_3_link'/>
@@ -71,4 +79,5 @@
         <xacro:call macro="${right_gripper_name}_col_with" prefix='right_gripper' link='right_camera_link'/>
     </xacro:if>
+    <!-- Define other groups -->
     <group name="left_arm">
         <chain base_link="left_base_link" tip_link="left_tool"/>
@@ -82,20 +91,4 @@
     </group>
     <!--GROUP STATES: Purpose: Define a named state for a particular group, in terms of joint values. This is useful to define states like 'folded arms'-->
-    <group_state name="open" group="left_gripper">
-        <joint name="left_gripper_joint" value="0.0"/>
-        <joint name="left_gripper_mirror_joint" value="0.0"/>
-    </group_state>
-    <group_state name="close" group="left_gripper">
-        <joint name="left_gripper_joint" value="1.3"/>
-        <joint name="left_gripper_mirror_joint" value="1.3"/>
-    </group_state>
-    <group_state name="open" group="right_gripper">
-        <joint name="right_gripper_joint" value="0.0"/>
-        <joint name="right_gripper_mirror_joint" value="0.0"/>
-    </group_state>
-    <group_state name="close" group="right_gripper">
-        <joint name="right_gripper_joint" value="1.3"/>
-        <joint name="right_gripper_mirror_joint" value="1.3"/>
-    </group_state>
     <group_state name="default" group="left_arm">
         <joint name="left_elbow_joint" value="-1.57"/>

Commit message: Add sim parameter in urdf/srdf for necessary variations

File: prl_ur5_description/urdf/_gripper.urdf.xacro (robot description, xacro)
@@ -3,5 +3,5 @@
   <!-- onrobot RG2(6) -->
   <xacro:include filename="$(find onrobot_description)/urdf/onrobot_rg.urdf.xacro"/>
-  <xacro:macro name="gripper" params="gripper prefix parent pose hardware_interface">
+  <xacro:macro name="gripper" params="gripper prefix parent pose hardware_interface gz_sim">
     <!-- check gripper type -->
     <xacro:unless value="${gripper in [None, 'onrobot-rg2', 'onrobot-rg6', 'onrobot-rg6-v2'] or gripper.startswith('custom:') or gripper.startswith('allegro-hand:')}">

File: prl_ur5_description/urdf/_ur5.urdf.xacro (robot description, xacro)
@@ -17,4 +17,5 @@
       hardware_interface
       sensors
+      gz_sim
       gripper:=None
       gripper_pose:=None
@@ -46,5 +47,5 @@
     <!-- gripper -->
     <xacro:unless value="${gripper is None}">
-      <xacro:gripper gripper="${gripper}" prefix='${prefix}' parent="${prefix}tool" pose="${gripper_pose}" hardware_interface="${hardware_interface}"/>
+      <xacro:gripper gripper="${gripper}" prefix='${prefix}' parent="${prefix}tool" pose="${gripper_pose}" hardware_interface="${hardware_interface}" gz_sim="${gz_sim}"/>
       <!-- Right angle connector -->
       <link name="${prefix}wrist_connector_link">

File: prl_ur5_description/urdf/prl_ur5.urdf.xacro (robot description, xacro)
@@ -5,5 +5,5 @@
   <!-- Fixed cameras -->
   <xacro:include filename="$(find prl_ur5_description)/urdf/_fixed_cameras.urdf.xacro"/>
-  <xacro:macro name="prl_ur5" params="setup_file hardware_interface sensors:=false table:=true backwall:=true ceiling:=true">
+  <xacro:macro name="prl_ur5" params="setup_file hardware_interface gz_sim sensors:=false table:=true backwall:=true ceiling:=true">
     <!-- base link -->
     <link name="prl_ur5_base"/>
@@ -118,5 +118,6 @@
                  camera="${left.get('camera')}"
                  camera_pose="${left.get('camera_pose')}"
-                 hardware_interface="${hardware_interface}"/>
+                 hardware_interface="${hardware_interface}"
+                 gz_sim="${gz_sim}"/>
     </xacro:if>
     <!-- right arm -->
@@ -133,5 +134,6 @@
                  camera="${right.get('camera')}"
                  camera_pose="${right.get('camera_pose')}"
-                 hardware_interface="${hardware_interface}"/>
+                 hardware_interface="${hardware_interface}"
+                 gz_sim="${gz_sim}"/>
     </xacro:if>
     <!-- head -->
@@ -146,26 +148,28 @@
     </xacro:if>
     <!-- gazebo stuff -->
-    <gazebo>
-      <!-- enable ros_control loop -->
-      <plugin name="ros_control_arms" filename="libgazebo_ros_control_select_joints.so">
-        <joints>
-          left_shoulder_pan_joint  right_shoulder_pan_joint
-          left_shoulder_lift_joint right_shoulder_lift_joint
-          left_elbow_joint         right_elbow_joint
-          left_wrist_1_joint       right_wrist_1_joint
-          left_wrist_2_joint       right_wrist_2_joint
-          left_wrist_3_joint       right_wrist_3_joint
-        </joints>
-      </plugin>
-      <!-- gravity compensation -->
-      <plugin name="gravity_compensation" filename="libGravityCompensationPlugin.so">
-        <uri>model://prl_ur5_robot</uri>
-      </plugin>
-      <!-- fix base in Gazebo -->
-      <joint name="fixed" type="fixed">
-        <parent>world</parent>
-        <child>prl_ur5_base</child>
-      </joint>
-    </gazebo>
+    <xacro:if value="${gz_sim}">
+      <gazebo>
+        <!-- enable ros_control loop -->
+        <plugin name="ros_control_arms" filename="libgazebo_ros_control_select_joints.so">
+          <joints>
+            left_shoulder_pan_joint  right_shoulder_pan_joint
+            left_shoulder_lift_joint right_shoulder_lift_joint
+            left_elbow_joint         right_elbow_joint
+            left_wrist_1_joint       right_wrist_1_joint
+            left_wrist_2_joint       right_wrist_2_joint
+            left_wrist_3_joint       right_wrist_3_joint
+          </joints>
+        </plugin>
+        <!-- gravity compensation -->
+        <plugin name="gravity_compensation" filename="libGravityCompensationPlugin.so">
+          <uri>model://prl_ur5_robot</uri>
+        </plugin>
+        <!-- fix base in Gazebo -->
+        <joint name="fixed" type="fixed">
+          <parent>world</parent>
+          <child>prl_ur5_base</child>
+        </joint>
+      </gazebo>
+    </xacro:if>
   </xacro:macro>
 </robot>

File: prl_ur5_description/urdf/prl_ur5_robot.urdf.xacro (robot description, xacro)
@@ -6,4 +6,5 @@
   <xacro:arg name="sensors" default="false"/>
   <xacro:arg name="hardware_interface" default="hardware_interface/PositionJointInterface"/>
+  <xacro:arg name="gz_sim" default="false"/>
   <!-- ur5 robot -->
   <xacro:include filename="$(find prl_ur5_description)/urdf/prl_ur5.urdf.xacro"/>
@@ -11,4 +12,5 @@
                  table="$(arg table)"
                  hardware_interface="$(arg hardware_interface)"
-                 sensors="$(arg sensors)"/>
+                 sensors="$(arg sensors)"
+                 gz_sim="$(arg gz_sim)"/>
 </robot>

Commit message: Add grasp_frame for allegro hand gripper

File: prl_ur5_description/urdf/_gripper.urdf.xacro (robot description, xacro)
@@ -32,4 +32,10 @@
         <origin xyz="${pose['x']} ${pose['y']} ${pose['z']}" rpy="${pose['roll']} ${pose['pitch']} ${pose['yaw']}"/>
       </xacro:allegro_hand>
+      <link name="${prefix}gripper_grasp_frame"/>
+      <joint name="${prefix}gripper_grasp_frame_joint" type="fixed">
+          <parent link="${prefix}gripper_palm_link"/>
+          <child link="${prefix}gripper_grasp_frame"/>
+          <origin rpy="0 0 0" xyz="0.05 0 -0.025"/>
+      </joint>
     </xacro:if>
     <!-- if custom gripper -->
