Commit message: Add backwall mesh in robot urdf to prevent collisions

File: prl_ur5_description/urdf/prl_ur5.urdf.xacro (robot description, xacro)
@@ -5,5 +5,5 @@
   <!-- gazebo -->
   <xacro:include filename="$(find prl_ur5_description)/urdf/prl_ur5.gazebo.xacro"/>
-  <xacro:macro name="prl_ur5" params="setup_file hardware_interface table:=true">
+  <xacro:macro name="prl_ur5" params="setup_file hardware_interface table:=true backwall:=true">
     <!-- base link -->
     <link name="prl_ur5_base"/>
@@ -56,4 +56,25 @@
       </joint>
     </xacro:if>
+    <!-- back wall -->
+    <xacro:if value="$(arg backwall)">
+      <link name="backwall_link">
+        <visual>
+          <geometry>
+            <box size="3 0.1 3" />
+          </geometry>
+          <material name="grey"><color rgba="0.8 0.8 0.8 0.2"/></material>
+        </visual>
+        <collision>
+          <geometry>
+            <box size="3 0.1 3" />
+          </geometry>
+        </collision>
+      </link>
+      <joint name="backwall_fix" type="fixed">
+        <parent link="prl_ur5_base"/>
+        <child link = "backwall_link"/>
+        <origin xyz="0 -1.05 0" rpy="0.0 0.0 0.0"/>
+      </joint>
+    </xacro:if>
     <!-- left arm -->
     <xacro:property name="left" value="${setup_file.get('left')}"/>

Commit message: Fix sim : change backwall size

File: prl_ur5_description/urdf/prl_ur5.urdf.xacro (robot description, xacro)
@@ -61,5 +61,5 @@
         <visual>
           <geometry>
-            <box size="3 0.1 3" />
+            <box size="3 0.1 2.5" />
           </geometry>
           <material name="grey"><color rgba="0.8 0.8 0.8 0.2"/></material>
@@ -67,5 +67,5 @@
         <collision>
           <geometry>
-            <box size="3 0.1 3" />
+            <box size="3 0.1 2.5" />
           </geometry>
         </collision>
@@ -74,5 +74,5 @@
         <parent link="prl_ur5_base"/>
         <child link = "backwall_link"/>
-        <origin xyz="0 -1.05 0" rpy="0.0 0.0 0.0"/>
+        <origin xyz="0 -1.05 0.5" rpy="0.0 0.0 0.0"/>
       </joint>
     </xacro:if>

Commit message: Update vention table geometries

File: prl_ur5_description/urdf/prl_ur5.urdf.xacro (robot description, xacro)
@@ -14,18 +14,11 @@
           <mesh filename="package://prl_ur5_description/model/vention_tower.dae"/>
         </geometry>
+        <material name="Cyan">
+  14        <color rgba="0 1.0 1.0 1.0"/>
+  15      </material>
       </visual>
       <collision>
         <geometry>
-          <mesh filename="package://prl_ur5_description/model/vention_tower_1.stl"/>
-        </geometry>
-      </collision>
-      <collision>
-        <geometry>
-          <mesh filename="package://prl_ur5_description/model/vention_tower_2.stl"/>
-        </geometry>
-      </collision>
-      <collision>
-        <geometry>
-          <mesh filename="package://prl_ur5_description/model/vention_tower_3.stl"/>
+          <mesh filename="package://prl_ur5_description/model/vention_tower.stl"/>
         </geometry>
       </collision>

Commit message: Add ceiling to urdf to bound motion

File: prl_ur5_description/urdf/prl_ur5.urdf.xacro (robot description, xacro)
@@ -7,5 +7,5 @@
   <!-- Fixed cameras -->
   <xacro:include filename="$(find prl_ur5_description)/urdf/_fixed_cameras.urdf.xacro"/>
-  <xacro:macro name="prl_ur5" params="setup_file hardware_interface table:=true backwall:=true">
+  <xacro:macro name="prl_ur5" params="setup_file hardware_interface table:=true backwall:=true ceiling:=true">
     <!-- base link -->
     <link name="prl_ur5_base"/>
@@ -76,4 +76,25 @@
       </joint>
     </xacro:if>
+    <!-- ceiling wall -->
+    <xacro:if value="$(arg ceiling)">
+      <link name="ceiling_link">
+        <visual>
+          <geometry>
+            <box size="3 1.95 0.1" />
+          </geometry>
+          <material name="grey"><color rgba="0.8 0.8 0.8 0.1"/></material>
+        </visual>
+        <collision>
+          <geometry>
+            <box size="3 1.95 0.1" />
+          </geometry>
+        </collision>
+      </link>
+      <joint name="ceiling_fix" type="fixed">
+        <parent link="prl_ur5_base"/>
+        <child link = "ceiling_link"/>
+        <origin xyz="0 0 1.3" rpy="0.0 0.0 0.0"/>
+      </joint>
+    </xacro:if>
     <!-- left arm -->
     <xacro:property name="left" value="${setup_file.get('left')}"/>

Commit message: Use gazebo_ros_control_select_joints and simplify gazebo config

File: prl_ur5_description/urdf/prl_ur5.urdf.xacro (robot description, xacro)
@@ -3,6 +3,4 @@
   <!-- single arm -->
   <xacro:include filename="$(find prl_ur5_description)/urdf/_ur5.urdf.xacro"/>
-  <!-- gazebo -->
-  <xacro:include filename="$(find prl_ur5_description)/urdf/prl_ur5.gazebo.xacro"/>
   <!-- Fixed cameras -->
   <xacro:include filename="$(find prl_ur5_description)/urdf/_fixed_cameras.urdf.xacro"/>
@@ -148,5 +146,26 @@
     </xacro:if>
     <!-- gazebo stuff -->
-    <xacro:prl_ur5_gazebo/>
+    <gazebo>
+      <!-- enable ros_control loop -->
+      <plugin name="ros_control_arms" filename="libgazebo_ros_control_select_joints.so">
+        <joints>
+          left_shoulder_pan_joint  right_shoulder_pan_joint
+          left_shoulder_lift_joint right_shoulder_lift_joint
+          left_elbow_joint         right_elbow_joint
+          left_wrist_1_joint       right_wrist_1_joint
+          left_wrist_2_joint       right_wrist_2_joint
+          left_wrist_3_joint       right_wrist_3_joint
+        </joints>
+      </plugin>
+      <!-- gravity compensation -->
+      <plugin name="gravity_compensation" filename="libGravityCompensationPlugin.so">
+        <uri>model://prl_ur5_robot</uri>
+      </plugin>
+      <!-- fix base in Gazebo -->
+      <joint name="fixed" type="fixed">
+        <parent>world</parent>
+        <child>prl_ur5_base</child>
+      </joint>
+    </gazebo>
   </xacro:macro>
 </robot>

Commit message: Update workbench mesh & update walls position

File: prl_ur5_description/urdf/prl_ur5.urdf.xacro (robot description, xacro)
@@ -5,44 +5,14 @@
   <!-- Fixed cameras -->
   <xacro:include filename="$(find prl_ur5_description)/urdf/_fixed_cameras.urdf.xacro"/>
-  <xacro:macro name="prl_ur5" params="setup_file hardware_interface gz_sim sensors:=false table:=true backwall:=true ceiling:=true">
+  <xacro:macro name="prl_ur5" params="setup_file hardware_interface gz_sim sensors:=false table:=true backwall:=true leftwall:=true">
     <!-- base link -->
     <link name="prl_ur5_base"/>
-    <!-- bimanual stand -->
-    <link name="stand_link">
-      <visual>
-        <geometry>
-          <mesh filename="package://prl_ur5_description/model/vention_tower.dae"/>
-        </geometry>
-        <material name="Cyan">
-          <color rgba="0 1.0 1.0 1.0"/>
-        </material>
-      </visual>
-      <collision>
-        <geometry>
-          <mesh filename="package://prl_ur5_description/model/vention_tower_bottom_convex.stl"/>
-        </geometry>
-      </collision>
-      <collision>
-        <geometry>
-          <mesh filename="package://prl_ur5_description/model/vention_tower_middle_convex.stl"/>
-        </geometry>
-      </collision>
-      <collision>
-        <geometry>
-          <mesh filename="package://prl_ur5_description/model/vention_tower_top_convex.stl"/>
-        </geometry>
-      </collision>
-    </link>
-    <joint name="stand_fix" type="fixed">
-      <parent link="prl_ur5_base"/>
-      <child link = "stand_link"/>
-      <origin xyz="0.0 -0.3825 0.0" rpy="0.0 0.0 0.0"/>
-    </joint>
     <!-- table -->
+    <!-- bimanual workbench -->
     <xacro:if value="$(arg table)">
       <link name="table_link">
         <visual>
           <geometry>
-            <mesh filename="package://prl_ur5_description/model/vention_table.dae"/>
+            <mesh filename="package://prl_ur5_description/model/vention_table.stl"/>
           </geometry>
         </visual>
@@ -53,9 +23,9 @@
         </collision>
       </link>
-      <joint name="table_fix" type="fixed">
-        <parent link="stand_link"/>
-        <child link = "table_link"/>
-        <origin xyz="0.0 0.0 0.0" rpy="0.0 0.0 0.0"/>
-      </joint>
+    <joint name="table_fix" type="fixed">
+      <parent link="prl_ur5_base"/>
+      <child link = "table_link"/>
+      <origin xyz="0.0 0.0 0.0" rpy="0.0 0.0 0.0"/>
+    </joint>
     </xacro:if>
     <!-- Cameras fixtures (if any) -->
@@ -68,5 +38,5 @@
         <visual>
           <geometry>
-            <box size="3 0.1 2.5" />
+            <box size="3.5 0.1 2" />
           </geometry>
           <material name="grey"><color rgba="0.8 0.8 0.8 0.2"/></material>
@@ -74,5 +44,5 @@
         <collision>
           <geometry>
-            <box size="3 0.1 2.5" />
+            <box size="3.5 0.1 2" />
           </geometry>
         </collision>
@@ -81,13 +51,13 @@
         <parent link="prl_ur5_base"/>
         <child link = "backwall_link"/>
-        <origin xyz="0 -1.05 0.5" rpy="0.0 0.0 0.0"/>
+        <origin xyz="0 -1.05 0.25" rpy="0.0 0.0 0.0"/>
       </joint>
     </xacro:if>
-    <!-- ceiling wall -->
-    <xacro:if value="$(arg ceiling)">
-      <link name="ceiling_link">
+    <!-- left wall -->
+    <xacro:if value="$(arg leftwall)">
+      <link name="leftwall_link">
         <visual>
           <geometry>
-            <box size="3 1.95 0.1" />
+            <box size="0.1 1.95 2" />
           </geometry>
           <material name="grey"><color rgba="0.8 0.8 0.8 0.1"/></material>
@@ -95,12 +65,12 @@
         <collision>
           <geometry>
-            <box size="3 1.95 0.1" />
+            <box size="0.1 1.95 2" />
           </geometry>
         </collision>
       </link>
-      <joint name="ceiling_fix" type="fixed">
+      <joint name="leftwall_fix" type="fixed">
         <parent link="prl_ur5_base"/>
-        <child link = "ceiling_link"/>
-        <origin xyz="0 0 1.3" rpy="0.0 0.0 0.0"/>
+        <child link = "leftwall_link"/>
+        <origin xyz="-1.65 0 0.25" rpy="0.0 0.0 0.0"/>
       </joint>
     </xacro:if>
@@ -109,5 +79,5 @@
     <xacro:if value="${left is not None}">
       <xacro:ur5 prefix="left_"
-                 parent="stand_link"
+                 parent="prl_ur5_base"
                  kinematics="$(find prl_ur5_robot_configuration)/config/${left['arm_kinematics']}"
                  joint_limits="$(find prl_ur5_robot_configuration)/config/${left['arm_joint_limits']}"
@@ -125,5 +95,5 @@
     <xacro:if value="${right is not None}">
       <xacro:ur5 prefix="right_"
-                 parent="stand_link"
+                 parent="prl_ur5_base"
                  kinematics="$(find prl_ur5_robot_configuration)/config/${right['arm_kinematics']}"
                  joint_limits="$(find prl_ur5_robot_configuration)/config/${right['arm_joint_limits']}"
@@ -136,14 +106,4 @@
                  hardware_interface="${hardware_interface}"
                  gz_sim="${gz_sim}"/>
-    </xacro:if>
-    <!-- head -->
-    <xacro:property name="head" value="${setup_file.get('head')}"/>
-    <xacro:if value="${head is not None}">
-      <xacro:unless value="${head.get('camera') is None}">
-        <xacro:camera_sensor prefix='head_'
-                             parent="stand_link"
-                             camera="${head['camera']}"
-                             pose="${head['camera_pose']}"/>
-      </xacro:unless>
     </xacro:if>
     <!-- gazebo stuff -->
